File: electrical/integration/main.sch (EAGLE design)
At the start: 0 parts

Commit message: replace caps
Other:
- note removed: "Breakout Connector"
- note removed: "If we neeed it, wire to 24V at motor controller"
